File: hardware/sensor_board/SensorBoard.kicad_sch (KiCad schematic)
At the start: 76 parts, among them J1 Relay Board Connector, J10 GND BUS, J11 FEED SENSOR R1, J12 Relay Pull, J13 SPARE GPIO, J15 LED L1, J16 LED L2, J17 LED L3, J18 LED L4, J19 LED R1, J2 Pi 5V, J20 EXT, J21 LED R2, J22 LED R3, J23 LED R4, J24 Raspberry Pi GPIO header, J25 RTC Header, J26 I2C0, J27 I2C1, J28 I2C2, J29 I2C3, J3 Display 5V, J30 I2C4, J31 I2C5, J32 I2C6, J33 I2C7, J4 DC IN 5V, J5 VSYS BUS, J6 FEED SENSOR L2, J7 3V3 BUS, J8 FEED SENSOR R2, J9 FEED SENSOR L1, Q1 PN2222A, Q2 PN2222A, Q3 PN2222A, Q4 PN2222A, Q5 PN2222A, Q6 PN2222A, Q7 PN2222A, Q8 PN2222A, SW1 Pico Reset, U1 Raspberry Pico, U2 74HC595, U3 TCA9548A, U4 LM1117, U5 DS3231MZ, U6 74HC165

Commit message: Board revisions 3.1 - added mutiple external switch connectors, clock battery sensing path to pico, jumpers to control feed sensor outputs and relay pulls
Parts:
- removed J10: GND BUS, Connector_PinHeader_2.54mm:PinHeader_1x03_P2.54mm_Vertical, symbol Connector_Generic:Conn_01x03
- removed J12: Relay Pull, Connector_PinHeader_2.54mm:PinHeader_1x03_P2.54mm_Vertical, symbol Connector_Generic:Conn_01x03
- removed J13: SPARE GPIO, Connector_PinHeader_2.54mm:PinHeader_1x02_P2.54mm_Vertical, symbol Connector_Generic:Conn_01x02
- removed J15: LED L1, Connector_JST:JST_XH_B2B-XH-A_1x02_P2.50mm_Vertical, symbol Connector_Generic:Conn_02x01
- removed J16: LED L2, Connector_JST:JST_XH_B2B-XH-A_1x02_P2.50mm_Vertical, symbol Connector_Generic:Conn_02x01
- removed J17: LED L3, Connector_JST:JST_XH_B2B-XH-A_1x02_P2.50mm_Vertical, symbol Connector_Generic:Conn_02x01
- removed J18: LED L4, Connector_JST:JST_XH_B2B-XH-A_1x02_P2.50mm_Vertical, symbol Connector_Generic:Conn_02x01
- removed J19: LED R1, Connector_JST:JST_XH_B2B-XH-A_1x02_P2.50mm_Vertical, symbol Connector_Generic:Conn_02x01
- removed J21: LED R2, Connector_JST:JST_XH_B2B-XH-A_1x02_P2.50mm_Vertical, symbol Connector_Generic:Conn_02x01
- removed J22: LED R3, Connector_JST:JST_XH_B2B-XH-A_1x02_P2.50mm_Vertical, symbol Connector_Generic:Conn_02x01
- removed J23: LED R4, Connector_JST:JST_XH_B2B-XH-A_1x02_P2.50mm_Vertical, symbol Connector_Generic:Conn_02x01
- removed J5: VSYS BUS, Connector_PinHeader_2.54mm:PinHeader_1x03_P2.54mm_Vertical, symbol Connector_Generic:Conn_01x03
- added J14: Left LEDs, Connector_JST:JST_XH_B5B-XH-A_1x05_P2.50mm_Vertical, symbol Connector_Generic:Conn_01x05
- added J15: Right LEDs, Connector_JST:JST_XH_B5B-XH-A_1x05_P2.50mm_Vertical, symbol Connector_Generic:Conn_01x05
- added J16: Reset, Connector_JST:JST_XH_B2B-XH-A_1x02_P2.50mm_Vertical, symbol Connector_Generic:Conn_01x02
- added J17: Shutdown, Connector_JST:JST_XH_B2B-XH-A_1x02_P2.50mm_Vertical, symbol Connector_Generic:Conn_01x02
- added JP1: Relay Pull, Connector_PinHeader_2.54mm:PinHeader_1x03_P2.54mm_Vertical, symbol Jumper:Jumper_3_Open
- added JP2: Feed Sensor Power, Connector_PinHeader_2.54mm:PinHeader_1x03_P2.54mm_Vertical, symbol Jumper:Jumper_3_Open
- added R10, R9: 10k, Resistor_THT:R_Axial_DIN0207_L6.3mm_D2.5mm_P7.62mm_Horizontal, symbol Device:R
- added R21, R22: 100k, Resistor_THT:R_Axial_DIN0207_L6.3mm_D2.5mm_P7.62mm_Horizontal, symbol Device:R
- J1: footprint Connector_PinHeader_2.54mm:PinHeader_1x10_P2.54mm_Vertical -> Connector_JST:JST_XH_B10B-XH-A_1x10_P2.50mm_Vertical
- J11: value FEED SENSOR R1 -> Feed Sensor R2
- J20: footprint Connector_JST:JST_XH_B8B-XH-A_1x08_P2.50mm_Vertical -> Connector_JST:JST_XH_B10B-XH-A_1x10_P2.50mm_Vertical; symbol Connector_Generic:Conn_01x08 -> Connector_Generic:Conn_01x10
- J4: value DC IN 5V -> DC 5V
- J6: value FEED SENSOR L2 -> Feed Sensor L1
- J7: value 3V3 BUS -> Power bus
- J8: value FEED SENSOR R2 -> Feed Sensor R1
- J9: value FEED SENSOR L1 -> Feed Sensor L2
Connections:
- net GPIO20 is gone; now on an unnamed net: U1.26 (GPIO20)
- net +3V3: now also JP2.1 (A); no longer J11.1 (Pin_1), J6.1 (Pin_1), J7.2 (Pin_2), J7.3 (Pin_3), J8.1 (Pin_1), J9.1 (Pin_1)
- net FEED SENSOR L1 DETECT: now also J6.4 (Pin_4), U1.1 (GPIO0); no longer J9.4 (Pin_4), U1.5 (GPIO3)
- net FEED SENSOR L1 RX: now also J6.5 (Pin_5), U1.7 (GPIO5); no longer J9.5 (Pin_5), U1.10 (GPIO7)
- net FEED SENSOR L1 TX: now also J6.2 (Pin_2), U1.6 (GPIO4); no longer J9.2 (Pin_2), U1.9 (GPIO6)
- net FEED SENSOR L2 DETECT: now also J9.4 (Pin_4), U1.2 (GPIO1); no longer J6.4 (Pin_4), U1.4 (GPIO2)
- net FEED SENSOR L2 RX: now also J9.5 (Pin_5), U1.10 (GPIO7); no longer J6.5 (Pin_5), U1.7 (GPIO5)
- net FEED SENSOR L2 TX: now also J9.2 (Pin_2), U1.9 (GPIO6); no longer J6.2 (Pin_2), U1.6 (GPIO4)
- net FEED SENSOR R1 DETECT: now also J8.4 (Pin_4), U1.4 (GPIO2); no longer J11.4 (Pin_4), U1.1 (GPIO0)
- net FEED SENSOR R1 RX: now also J8.5 (Pin_5), U1.34 (GPIO28_ADC2); no longer J11.5 (Pin_5), U1.29 (GPIO22)
- net FEED SENSOR R1 TX: now also J8.2 (Pin_2), U1.32 (GPIO27_ADC1); no longer J11.2 (Pin_2), U1.31 (GPIO26_ADC0)
- net FEED SENSOR R2 DETECT: now also J11.4 (Pin_4), U1.5 (GPIO3); no longer J8.4 (Pin_4), U1.2 (GPIO1)
- net FEED SENSOR R2 RX: now also J11.5 (Pin_5), U1.29 (GPIO22); no longer J8.5 (Pin_5), U1.32 (GPIO27_ADC1)
- net FEED SENSOR R2 TX: now also J11.2 (Pin_2), U1.27 (GPIO21); no longer J8.2 (Pin_2), U1.34 (GPIO28_ADC2)
- net GND: now also J1.9 (Pin_9), J20.9 (Pin_9), J7.2 (Pin_2), U1.33 (AGND), J14.1 (Pin_1), J15.1 (Pin_1), J16.1 (Pin_1), J17.1 (Pin_1), JP1.3 (B), R22.1; no longer J1.1 (Pin_1)
- net VS: now also J7.3 (Pin_3), JP1.1 (A), JP2.3 (B)
- net at Q6.3 (C), RN2.7 (R6): now also J1.6 (Pin_6); no longer J1.7 (Pin_7)
- net at R11.2: now also J14.2 (Pin_2)
- net at Q1.3 (C), RN2.2 (R1): now also J1.1 (Pin_1); no longer J1.2 (Pin_2)
- net at R12.2: now also J14.3 (Pin_3)
- net at RN2.1 (common): now also JP1.2 (C)
- net at Q2.3 (C), RN2.3 (R2): now also J1.2 (Pin_2); no longer J1.3 (Pin_3)
- net at Q3.3 (C), RN2.4 (R3): now also J1.3 (Pin_3); no longer J1.4 (Pin_4)
- net at Q4.3 (C), RN2.5 (R4): now also J1.4 (Pin_4); no longer J1.5 (Pin_5)
- net at Q5.3 (C), RN2.6 (R5): now also J1.5 (Pin_5); no longer J1.6 (Pin_6)
- net at Q7.3 (C), RN2.8 (R7): now also J1.7 (Pin_7); no longer J1.8 (Pin_8)
- net at Q8.3 (C), RN2.9 (R8): now also J1.8 (Pin_8); no longer J1.9 (Pin_9)
- net at BT1.1 (+), U5.6 (VBAT): now also R21.2
- net at R18.2: now also J15.5 (Pin_5)
- net at U6.1 (~{PL}): no longer U1.27 (GPIO21)
- net at R13.2: now also J14.4 (Pin_4)
- net at R17.2: now also J15.4 (Pin_4)
- net at C2.1, J24.1 (3V3), J25.5 (Pin_5)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: now also R10.1, R9.2
- net at R14.2: now also J14.5 (Pin_5)
- net at J24.11 (GPIO17): now also J16.2 (Pin_2), R9.1
- net at J24.7 (GCLK0/GPIO4): now also J17.2 (Pin_2), R10.2
- net at R15.2: now also J15.2 (Pin_2)
- net RST: now reaches SW1.2, U1.30 (RUN)
- net RST: now also J20.10 (Pin_10)
- net at R16.2: now also J15.3 (Pin_3)
- net GPIO19: no longer names the net of U1.25 (GPIO19)
- new net: J11.1 (Pin_1), J6.1 (Pin_1), J8.1 (Pin_1), J9.1 (Pin_1), JP2.2 (C)
- new net: R21.1, R22.2, U1.31 (GPIO26_ADC0)
- no-connect marks 35 -> 33
Other:
- moved on the sheet: BT1, C1, C2, C3, C4, C5, D1, D2, J1, J11, J2, J24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
