File: hardware/PCB/HardwareInterfaceBoard.kicad_sch (KiCad schematic)
At the start: 81 parts, among them J1 Relay Board Connector, J11 Feed Sensor R2, J14 Left LEDs, J15 Right LEDs, J16 Reset, J17 Shutdown, J2 Pi 5V, J20 EXT, J24 Raspberry Pi GPIO header, J25 RTC Header, J26 I2C0, J27 I2C1, J28 I2C2, J29 I2C3, J3 Display 5V, J30 I2C4, J31 I2C5, J32 I2C6, J33 I2C7, J4 DC 5V, J5 GPIO, J6 Feed Sensor L1, J7 Power bus, J8 Feed Sensor R1, J9 Feed Sensor L2, Q1 PN2222A, Q2 PN2222A, Q3 PN2222A, Q4 PN2222A, Q5 PN2222A, Q6 PN2222A, Q7 PN2222A, Q8 PN2222A, Q9 TP0610L, SW1 Pico Reset, U1 Raspberry Pico, U2 74HC595, U3 TCA9548A, U4 LM1117, U5 DS3231MZ, U6 74HC165, U7 74HC165

Commit message: Added in some badly set resistor values
Parts:
- R11, R12, R13: value R1 -> 300
- R14: value R2 -> 300
- R15: value R3 -> 300
- R16: value R4 -> 300
- R17: value R5 -> 300
- R18: value R6 -> 300
Changed lines of the file:
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@@
     (in_bom yes) (on_board yes)
     (property "Reference" "R11" (id 0) (at 359.41 283.21 90))
-    (property "Value" "R1" (id 1) (at 360.6799 280.67 0)
+    (property "Value" "300" (id 1) (at 360.6799 280.67 0)
       (effects (font (size 1.27 1.27)) (justify left) hide)
     )
@@
     (in_bom yes) (on_board yes)
     (property "Reference" "R18" (id 0) (at 359.41 300.99 90))
-    (property "Value" "R6" (id 1) (at 360.6799 298.45 0)
+    (property "Value" "300" (id 1) (at 360.6799 298.45 0)
       (effects (font (size 1.27 1.27)) (justify left) hide)
     )
@@
     (in_bom yes) (on_board yes)
     (property "Reference" "R17" (id 0) (at 359.41 298.45 90))
-    (property "Value" "R5" (id 1) (at 360.6799 295.91 0)
+    (property "Value" "300" (id 1) (at 360.6799 295.91 0)
       (effects (font (size 1.27 1.27)) (justify left) hide)
     )
@@
     (in_bom yes) (on_board yes)
     (property "Reference" "R12" (id 0) (at 359.41 285.75 90))
-    (property "Value" "R1" (id 1) (at 360.6799 283.21 0)
+    (property "Value" "300" (id 1) (at 360.6799 283.21 0)
       (effects (font (size 1.27 1.27)) (justify left) hide)
     )
@@
     (in_bom yes) (on_board yes)
     (property "Reference" "R14" (id 0) (at 359.41 290.83 90))
-    (property "Value" "R2" (id 1) (at 360.6799 288.29 0)
+    (property "Value" "300" (id 1) (at 360.6799 288.29 0)
       (effects (font (size 1.27 1.27)) (justify left) hide)
     )
@@
     (in_bom yes) (on_board yes)
     (property "Reference" "R15" (id 0) (at 359.41 293.37 90))
-    (property "Value" "R3" (id 1) (at 360.6799 290.83 0)
+    (property "Value" "300" (id 1) (at 360.6799 290.83 0)
       (effects (font (size 1.27 1.27)) (justify left) hide)
     )
@@
     (in_bom yes) (on_board yes)
     (property "Reference" "R13" (id 0) (at 359.41 288.29 90))
-    (property "Value" "R1" (id 1) (at 360.6799 285.75 0)
+    (property "Value" "300" (id 1) (at 360.6799 285.75 0)
       (effects (font (size 1.27 1.27)) (justify left) hide)
     )
@@
     (in_bom yes) (on_board yes)
     (property "Reference" "R16" (id 0) (at 359.41 295.91 90))
-    (property "Value" "R4" (id 1) (at 360.6799 293.37 0)
+    (property "Value" "300" (id 1) (at 360.6799 293.37 0)
       (effects (font (size 1.27 1.27)) (justify left) hide)
     )
@@
     )
     (path "/0d4fc274-896e-42b8-8aaf-c5f954d38940"
-      (reference "R11") (unit 1) (value "R1") (footprint "Resistor_THT:R_Axial_DIN0207_L6.3mm_D2.5mm_P7.62mm_Horizontal")
+      (reference "R11") (unit 1) (value "300") (footprint "Resistor_THT:R_Axial_DIN0207_L6.3mm_D2.5mm_P7.62mm_Horizontal")
     )
     (path "/63e2acfb-22a6-48d2-961e-2f17c3003576"
-      (reference "R12") (unit 1) (value "R1") (footprint "Resistor_THT:R_Axial_DIN0207_L6.3mm_D2.5mm_P7.62mm_Horizontal")
+      (reference "R12") (unit 1) (value "300") (footprint "Resistor_THT:R_Axial_DIN0207_L6.3mm_D2.5mm_P7.62mm_Horizontal")
     )
     (path "/ccf7ec90-24de-45b6-8992-65368a1892eb"
-      (reference "R13") (unit 1) (value "R1") (footprint "Resistor_THT:R_Axial_DIN0207_L6.3mm_D2.5mm_P7.62mm_Horizontal")
+      (reference "R13") (unit 1) (value "300") (footprint "Resistor_THT:R_Axial_DIN0207_L6.3mm_D2.5mm_P7.62mm_Horizontal")
     )
     (path "/6f1ec6ff-882f-4606-9375-f252d2869ef6"
-      (reference "R14") (unit 1) (value "R2") (footprint "Resistor_THT:R_Axial_DIN0207_L6.3mm_D2.5mm_P7.62mm_Horizontal")
+      (reference "R14") (unit 1) (value "300") (footprint "Resistor_THT:R_Axial_DIN0207_L6.3mm_D2.5mm_P7.62mm_Horizontal")
     )
     (path "/8b3bfaaa-0e97-41e9-a52b-053852b9514d"
-      (reference "R15") (unit 1) (value "R3") (footprint "Resistor_THT:R_Axial_DIN0207_L6.3mm_D2.5mm_P7.62mm_Horizontal")
+      (reference "R15") (unit 1) (value "300") (footprint "Resistor_THT:R_Axial_DIN0207_L6.3mm_D2.5mm_P7.62mm_Horizontal")
     )
     (path "/eaf8655f-6d97-46b0-b14d-3b0d49ce8179"
-      (reference "R16") (unit 1) (value "R4") (footprint "Resistor_THT:R_Axial_DIN0207_L6.3mm_D2.5mm_P7.62mm_Horizontal")
+      (reference "R16") (unit 1) (value "300") (footprint "Resistor_THT:R_Axial_DIN0207_L6.3mm_D2.5mm_P7.62mm_Horizontal")
     )
     (path "/51fb5001-86c0-44ac-b688-35bddc35e6fe"
-      (reference "R17") (unit 1) (value "R5") (footprint "Resistor_THT:R_Axial_DIN0207_L6.3mm_D2.5mm_P7.62mm_Horizontal")
+      (reference "R17") (unit 1) (value "300") (footprint "Resistor_THT:R_Axial_DIN0207_L6.3mm_D2.5mm_P7.62mm_Horizontal")
     )
     (path "/2d676d3c-d776-4a26-af99-5ba5959832ff"
-      (reference "R18") (unit 1) (value "R6") (footprint "Resistor_THT:R_Axial_DIN0207_L6.3mm_D2.5mm_P7.62mm_Horizontal")
+      (reference "R18") (unit 1) (value "300") (footprint "Resistor_THT:R_Axial_DIN0207_L6.3mm_D2.5mm_P7.62mm_Horizontal")
     )
     (path "/b335ffa7-cd6c-4361-8681-d493a5ca4711"
